File: 02.POWER_SUPPLY_BB/02.POWER_SUPPLY_BB/02.POWER_SUPPLY_BB.kicad_sch (KiCad schematic)
At the start: 0 parts

Commit message: POWER_SUPPLY_BB - EESCHEMA - SYMBOL
Parts:
- added C1: 10u, symbol Device:C
- added C2: 0.1u, symbol Device:C
- added C3: 1u, symbol Device:C
- added D1: LED, symbol Device:LED
- added J1, J2: Conn_01x02_Pin, symbol Connector:Conn_01x02_Pin
- added J3, J4: Conn_01x03_Pin, symbol Connector:Conn_01x03_Pin
- added J5: Screw_Terminal_01x02, symbol Connector:Screw_Terminal_01x02
- added J6: Barrel_Jack_Switch, symbol Connector:Barrel_Jack_Switch
- added R1, R2: 330, symbol Device:R
- added R3: 560, symbol Device:R
- added S1: EG1218, digikey-footprints:Switch_Slide_11.6x4mm_EG1218, symbol dk_Slide-Switches:EG1218
- added U1: LM7806_TO220, Package_TO_SOT_THT:TO-220-3_Vertical, symbol Regulator_Linear:LM7806_TO220
- added U2: LM317_TO-220, Package_TO_SOT_THT:TO-220-3_Vertical, symbol Regulator_Linear:LM317_TO-220

Commit message: POWER_SUPPLY_BB - EESCHEMA - ARRANGE,ANNOTATE
Parts:
- added J7: Screw_Terminal_01x02, symbol Connector:Screw_Terminal_01x02
Other:
- moved on the sheet: C1, C2, C3, D1, J1, J2, J3, J4, J5, J6, R1, R2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

Commit message: POWER_SUPPLY_BB - EESCHEMA - ASSOCIATE
Parts:
- C1, C2, C3: footprint (none) -> Capacitor_THT:C_Disc_D3.0mm_W1.6mm_P2.50mm
- D1: footprint (none) -> LED_THT:LED_D5.0mm
- J1, J2: footprint (none) -> Connector_PinHeader_2.54mm:PinHeader_1x02_P2.54mm_Vertical
- J3, J4: footprint (none) -> Connector_PinHeader_2.54mm:PinHeader_1x03_P2.54mm_Vertical
- J5, J7: footprint (none) -> TerminalBlock:TerminalBlock_bornier-2_P5.08mm
- J6: footprint (none) -> Connector_BarrelJack:BarrelJack_Horizontal
- R1, R2, R3: footprint (none) -> Resistor_THT:R_Axial_DIN0204_L3.6mm_D1.6mm_P7.62mm_Horizontal
Changed lines of the file:
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@@
 			)
 		)
-		(property "Footprint" ""
+		(property "Footprint" "Capacitor_THT:C_Disc_D3.0mm_W1.6mm_P2.50mm"
 			(at 125.4252 76.2 0)
 			(effects
@@
 			)
 		)
-		(property "Footprint" ""
+		(property "Footprint" "Resistor_THT:R_Axial_DIN0204_L3.6mm_D1.6mm_P7.62mm_Horizontal"
 			(at 89.662 139.7 90)
 			(effects
@@
 			)
 		)
-		(property "Footprint" ""
+		(property "Footprint" "LED_THT:LED_D5.0mm"
 			(at 74.93 135.89 0)
 			(effects
@@
 			)
 		)
-		(property "Footprint" ""
+		(property "Footprint" "Resistor_THT:R_Axial_DIN0204_L3.6mm_D1.6mm_P7.62mm_Horizontal"
 			(at 89.662 115.57 90)
 			(effects
@@
 			)
 		)
-		(property "Footprint" ""
+		(property "Footprint" "Capacitor_THT:C_Disc_D3.0mm_W1.6mm_P2.50mm"
 			(at 79.7052 76.2 0)
 			(effects
@@
 			)
 		)
-		(property "Footprint" ""
+		(property "Footprint" "Resistor_THT:R_Axial_DIN0204_L3.6mm_D1.6mm_P7.62mm_Horizontal"
 			(at 50.292 128.27 90)
 			(effects
@@
 			)
 		)
-		(property "Footprint" ""
+		(property "Footprint" "TerminalBlock:TerminalBlock_bornier-2_P5.08mm"
 			(at 223.52 132.08 0)
 			(effects
@@
 			)
 		)
-		(property "Footprint" ""
+		(property "Footprint" "Connector_PinHeader_2.54mm:PinHeader_1x03_P2.54mm_Vertical"
 			(at 218.44 55.88 0)
 			(effects
@@
 			)
 		)
-		(property "Footprint" ""
+		(property "Footprint" "Connector_BarrelJack:BarrelJack_Horizontal"
 			(at 29.21 70.866 0)
 			(effects
@@
 			)
 		)
-		(property "Footprint" ""
+		(property "Footprint" "Connector_PinHeader_2.54mm:PinHeader_1x02_P2.54mm_Vertical"
 			(at 219.71 121.92 0)
 			(effects
@@
 			)
 		)
-		(property "Footprint" ""
+		(property "Footprint" "TerminalBlock:TerminalBlock_bornier-2_P5.08mm"
 			(at 222.25 81.28 0)
 			(effects
@@
 			)
 		)
-		(property "Footprint" ""
+		(property "Footprint" "Capacitor_THT:C_Disc_D3.0mm_W1.6mm_P2.50mm"
 			(at 107.6452 120.65 0)
 			(effects
@@
 			)
 		)
-		(property "Footprint" ""
+		(property "Footprint" "Connector_PinHeader_2.54mm:PinHeader_1x02_P2.54mm_Vertical"
 			(at 218.44 72.39 0)
 			(effects
@@
 			)
 		)
-		(property "Footprint" ""
+		(property "Footprint" "Connector_PinHeader_2.54mm:PinHeader_1x03_P2.54mm_Vertical"
 			(at 219.71 107.95 0)
 			(effects

Commit message: POWER_SUPPLY_BB - EESCHEMA - WIRING
Connections:
- net 5V: now reaches C2.1
- net 5V: now also J3.3 (Pin_3), J4.3 (Pin_3), U1.3 (VO)
- net GND: now reaches C2.2
- net GND: now also C1.2, C3.2, D1.1 (K), J1.1 (Pin_1), J2.1 (Pin_1), J5.1 (Pin_1), J6.2, J6.3, J7.1 (Pin_1), R3.2, U1.2 (GND)
- net at R3.1: now also R1.2, U2.1 (ADJ)
- net at D1.2 (A): now also R2.2
- net 3.3v: now reaches R1.1
- net 3.3v: now also C3.1, J3.1 (Pin_1), J4.1 (Pin_1), U2.2 (VO)
- net 12V: now reaches U2.3 (VI)
- net 12V: now also C1.1, R2.1, S1.1, U1.1 (VI)
- net at J7.2 (Pin_2): now also J2.2 (Pin_2), J4.2 (Pin_2)
- net at J3.2 (Pin_2): now also J1.2 (Pin_2), J5.2 (Pin_2)
- net at S1.2: now also J6.1
- no-connect marks 0 -> 1
Other:
- moved on the sheet: C1, C2, C3, D1, J1, J3, J5, J6, R1, R2, R3, S1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

Commit message: POWER_SUPPLY_BB - EESCHEMA - NET
Connections:
- net PWR_output: now reaches J2.2 (Pin_2), J4.2 (Pin_2), J7.2 (Pin_2)
- net PWR_output: now also J1.2 (Pin_2), J3.2 (Pin_2), J5.2 (Pin_2)
- net PWR_input: now reaches J6.1, S1.2
Changed lines of the file:
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@@
+		)
+	)
+	(label "PWR_output"
+		(at 177.8 116.84 0)
+		(effects
+			(font
+				(size 1.27 1.27)
+			)
+			(justify left bottom)
 		)
 	)
@@
 		)
 	)
+	(label "PWR_input"
+		(at 45.72 71.12 0)
+		(effects
+			(font
+				(size 1.27 1.27)
+			)
+			(justify left bottom)
+		)
+	)
+	(label "PWR_output"
+		(at 176.53 63.5 0)
+		(effects
+			(font
+				(size 1.27 1.27)
+			)
+			(justify left bottom)
+		)
+	)

Commit message: POWER_SUPPLY_BB - EESCHEMA - COMMENTS
Other:
- note added: "3.3v Circuit"
- note added: "Input and 5V circuit"
- note added: "Output and Switches"
Changed lines of the file:
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@@
 		(company "Gobal Krishnan")
+	)
+	(rectangle
+		(start 25.4 101.6)
+		(end 127 152.4)
+		(stroke
+			(width 0)
+			(type default)
+		)
+		(fill
+			(type none)
+		)
+	)
+	(rectangle
+		(start 160.02 50.8)
+		(end 213.36 153.035)
+		(stroke
+			(width 0)
+			(type default)
+		)
+		(fill
+			(type none)
+		)
+	)
+	(rectangle
+		(start 25.4 58.42)
+		(end 137.16 94.615)
+		(stroke
+			(width 0)
+			(type default)
+		)
+		(fill
+			(type none)
+		)
+	)
+	(text "3.3v Circuit"
+		(exclude_from_sim no)
+		(at 30.988 100.33 0)
+		(effects
+			(font
+				(size 1.27 1.27)
+			)
+		)
+	)
+	(text "Output and Switches"
+		(exclude_from_sim no)
+		(at 169.672 49.276 0)
+		(effects
+			(font
+				(size 1.27 1.27)
+			)
+		)
+	)
+	(text "Input and 5V circuit"
+		(exclude_from_sim no)
+		(at 34.798 57.15 0)
+		(effects
+			(font
+				(size 1.27 1.27)
+			)
+		)
 	)
 	(junction
