File: 03.EEPROM/EEPROM/EEPROM.kicad_sch (KiCad schematic)
At the start: 25 parts, among them U1 24LC1025, U2 DS1337S_, U3 24LC1025, U4 ATMEGA328P-AU, Y1 32.728 KHz, Y2 16 MHz

Commit message: EEPROM - EESCHEMA - COMMENT
Other:
- note added: "CLOCK"
- note added: "EEPROM"
- note added: "MCU"
- note added: "MOUNTING"
Changed lines of the file:
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@@
 		(company "Gobal Krishnan V")
+	)
+	(rectangle
+		(start 223.52 119.38)
+		(end 248.92 154.94)
+		(stroke
+			(width 0)
+			(type default)
+		)
+		(fill
+			(type none)
+		)
+	)
+	(rectangle
+		(start 25.4 119.38)
+		(end 127 160.02)
+		(stroke
+			(width 0)
+			(type default)
+		)
+		(fill
+			(type none)
+		)
+	)
+	(rectangle
+		(start 17.78 33.02)
+		(end 127 93.98)
+		(stroke
+			(width 0)
+			(type default)
+		)
+		(fill
+			(type none)
+		)
+	)
+	(rectangle
+		(start 137.16 33.02)
+		(end 259.08 109.22)
+		(stroke
+			(width 0)
+			(type default)
+		)
+		(fill
+			(type none)
+		)
+	)
+	(text "EEPROM"
+		(exclude_from_sim no)
+		(at 28.702 118.11 0)
+		(effects
+			(font
+				(size 1.27 1.27)
+			)
+		)
+	)
+	(text "MOUNTING"
+		(exclude_from_sim no)
+		(at 228.346 117.856 0)
+		(effects
+			(font
+				(size 1.27 1.27)
+			)
+		)
+	)
+	(text "CLOCK"
+		(exclude_from_sim no)
+		(at 20.828 31.75 0)
+		(effects
+			(font
+				(size 1.27 1.27)
+			)
+		)
+	)
+	(text "MCU"
+		(exclude_from_sim no)
+		(at 138.938 31.242 0)
+		(effects
+			(font
+				(size 1.27 1.27)
+			)
+		)
 	)
 	(junction
